Commit message: visual information from urdf is not needed for inverse kinematics computation

File: sunriseRobot/app_SunriseRobot/urdf/arm.urdf (robot description, URDF)
Before this commit: robot arm, 6 links, 5 joints
Links:
- link base_link: geometry 
- link link1: geometry 
- link link2: geometry 
- link link3: geometry 
- link link4: geometry 
- link link5: geometry 
